Commit message: Lidar/Imu

File: description/robot.urdf.xacro (robot description, xacro)
@@ -1,4 +1,5 @@
 <?xml version="1.0"?>
-<robot xmlns:xacro="http://www.ros.org/wiki/xacro"  name="robot">
-    <xacro:include filename="robot_core.xacro" />
+<robot xmlns:xacro="http://www.ros.org/wiki/xacro" name="robot">
+    <xacro:include filename="robot_core.xacro"/>
+    <xacro:include filename="robot_gazebo.xacro"/>
 </robot>

File: description/robot_core.xacro (robot description, xacro)
@@ -35,18 +35,4 @@
         </inertial>
     </link>
-    <!-- PLUGIN CORRIGIDO PARA GAZEBO HARMONIC -->
-    <gazebo>
-        <plugin name="gz::sim::systems::DiffDrive" filename="gz-sim-diff-drive-system">
-            <topic>/cmd_vel</topic>
-            <left_joint>left_wheel_joint</left_joint>
-            <right_joint>right_wheel_joint</right_joint>
-            <wheel_separation>0.35</wheel_separation>
-            <wheel_radius>0.05</wheel_radius>
-            <odom_topic>/odom</odom_topic>
-            <frame_id>odom</frame_id>
-            <child_frame_id>base_link</child_frame_id>
-            <odom_publish_frequency>30</odom_publish_frequency>
-        </plugin>
-    </gazebo>
     <!-- CHASSIS LINK -->
     <joint name="chassis_joint" type="fixed">
@@ -141,4 +127,12 @@
         </xacro:inertial_sphere>
     </link>
+    <!-- STEP 8 - IMU -->
+    <joint name="imu_joint" type="fixed">
+        <origin xyz="0 0 0" rpy="0 0 0" />
+        <parent link="base_link"/>
+        <child link="imu_link" />
+    </joint>
+    <link name="imu_link">
+    </link>
     <!-- STEP 10 - Lidar -->
     <joint type="fixed" name="scan_joint">
@@ -163,42 +157,7 @@
             <origin xyz="0 0 0.05" rpy="0 0 0"/>
             <geometry>
-                <mesh filename="/home/brunotavares/infinity_ws/src/infinity_bot/meshes/lidar.dae"/>
+                <mesh filename="model://meshes/lidar.dae" scale="2 2 2"/>
             </geometry>
         </visual>
     </link>
-    <gazebo reference="scan_link">
-        <sensor name="gpu_lidar" type="gpu_lidar">
-            <update_rate>10</update_rate>
-            <topic>scan</topic>
-            <gz_frame_id>scan_link</gz_frame_id>
-            <lidar>
-                <scan>
-                    <horizontal>
-                        <samples>720</samples>
-                        <resolution>1</resolution>
-                        <min_angle>-3.14156</min_angle>
-                        <max_angle>3.14156</max_angle>
-                    </horizontal>
-                    <vertical>
-                        <samples>3</samples>
-                        <min_angle>-0.001</min_angle>
-                        <max_angle>0.001</max_angle>
-                    </vertical>
-                </scan>
-                <range>
-                    <min>0.05</min>
-                    <max>10.0</max>
-                    <resolution>0.01</resolution>
-                </range>
-                <noise>
-                    <type>gaussian</type>
-                    <mean>0.0</mean>
-                    <stddev>0.01</stddev>
-                </noise>
-                <frame_id>scan_link</frame_id>
-            </lidar>
-            <always_on>1</always_on>
-            <visualize>true</visualize>
-        </sensor>
-    </gazebo>
 </robot>
